File: UINIO-MCU-GD32F103CBT6.kicad_pcb (KiCad board)
At the start: 2 copper layers, 68.4 x 20.3 mm, 43 parts, among them J1 Conn_01x24_Pin, J2 Conn_01x24_Pin, J3 Conn_01x04_Pin, SW1 BOOT1, SW2 NRST, SW3 BOOT0, U1 ME6211C33M5G-N, U2 GD32F103C8T6, Y1 32.768KHz, Y2 8MHz

Commit message: Release UINIO-MCU-GD32F103CBT6 version 3.1.0.
Other:
- board text added: "UINIO-MCU-GD32F103CBT6"
- board text added: "Version 3.1.0"
- board text removed: "UINIO-MCU-GD32F103C"
- board text removed: "Version 3.0.0"

Commit message: Update README.md.
Parts:
- removed ? (x2): LOGO, LOGO
Other:
- board text added: "Version 3.1.1"
- board text removed: "Version 3.1.0"

Commit message: Release UINIO-MCU-GD32F103CBT6 version 3.1.2.
Other:
- board text added: "Version 3.1.2"
- board text removed: "Version 3.1.1"
