File: UINIO-MCU-GD32F103CBT6.kicad_sch (KiCad schematic)
At the start: 37 parts, among them J1 Conn_01x24_Pin, J2 Conn_01x24_Pin, J3 Conn_01x04_Pin, SW1 BOOT1, SW2 NRST, SW3 BOOT0, U1 ME6211C33M5G-N, U2 GD32F103C8T6, Y1 32.768KHz, Y2 8MHz

Commit message: Release UINIO-MCU-GD32F103CBT6 version 3.1.0.
Other:
- title: UINIO-MCU-GD32F103C -> UINIO-MCU-GD32F103CBT6

Commit message: Update README.md.
Other:
- company: 电子技术博客 UinIO.com -> UinIO.com 电子技术工作室
- moved on the sheet: C12, J1, J2, R7, R8
